Commit message: added pickrobot urdf

File: pickbot_ws/install/pickbot_description/share/pickbot_description/urdf/pickbot.urdf.xacro (robot description, xacro)
@@ -1,4 +1,7 @@
 <?xml version="1.0"?>
 <robot xmlns:xacro="http://www.ros.org/wiki/xacro" name="pickbot">
+    <xacro:property name="PI" value="3.14159"/>
+    <xacro:property name="effort" value="30.0"/>
+    <xacro:property name="velocity" value="10.0"/>
     <link name="world"/>
     <link name="base_link">
@@ -15,3 +18,92 @@
         <origin rpy="0 0 0" xyz="0 0 0"/>
     </joint>
+    <link name="base_plate">
+        <visual>
+            <origin rpy="0 0 0" xyz="-0.39 -0.39 -0.56"/>
+            <geometry>
+                <mesh filename="package://pickbot_description/meshes/base_plate.STL" scale="0.01 0.01 0.01"/>
+            </geometry>
+        </visual>
+    </link>
+    <joint name="joint_1" type="revolute">
+        <parent link="base_link"/>
+        <child link="base_plate"/>
+        <axis xyz="0 0 1"/>
+        <origin rpy="0 0 0" xyz="0 0 0.307"/>
+        <limit lower="-${PI/2}" upper="${PI/2}" effort="${effort}" velocity="${velocity}"/>
+    </joint>
+    <link name="forward_drive_arm">
+        <visual>
+            <origin rpy="0 -${PI/2} ${PI/2}" xyz="0.19 0.06 -0.08"/>
+            <geometry>
+                <mesh filename="package://pickbot_description/meshes/forward_drive_arm.STL" scale="0.01 0.01 0.01"/>
+            </geometry>
+        </visual>
+    </link>
+    <joint name="joint_2" type="revolute">
+        <parent link="base_plate"/>
+        <child link="forward_drive_arm"/>
+        <axis xyz="1 0 0"/>
+        <origin rpy="0 0 0" xyz="-0.02 0 0.35"/>
+        <limit lower="-${PI/2}" upper="${PI/2}" effort="${effort}" velocity="${velocity}"/>
+    </joint>
+    <link name="horizontal_arm">
+        <visual>
+            <origin rpy="${PI/2} 0 ${PI/2}" xyz="-0.03 -0.4 -0.06"/>
+            <geometry>
+                <mesh filename="package://pickbot_description/meshes/horizontal_arm.STL" scale="0.01 0.01 0.01"/>
+            </geometry>
+        </visual>
+    </link>
+    <joint name="joint_3" type="revolute">
+        <parent link="forward_drive_arm"/>
+        <child link="horizontal_arm"/>
+        <axis xyz="1 0 0"/>
+        <origin rpy="0 0 0" xyz="0 0 0.8"/>
+        <limit lower="-${PI/2}" upper="${PI/2}" effort="${effort}" velocity="${velocity}"/>
+    </joint>
+    <link name="claw_support">
+        <visual>
+            <origin rpy="0 0 ${PI/2}" xyz="0 -0.05 -0.15"/>
+            <geometry>
+                <mesh filename="package://pickbot_description/meshes/claw_support.STL" scale="0.01 0.01 0.01"/>
+            </geometry>
+        </visual>
+    </link>
+    <joint name="horizontal_arm_to_claw_support" type="fixed">
+        <parent link="horizontal_arm"/>
+        <child link="claw_support"/>
+        <origin rpy="0 0 0" xyz="0 0.82 0"/>
+    </joint>
+    <link name="gripper_right">
+        <visual>
+            <origin rpy="0 0 -${PI/2}" xyz="-0.1 0.5 -0.1"/>
+            <geometry>
+                <mesh filename="package://pickbot_description/meshes/right_finger.STL" scale="0.01 0.01 0.01"/>
+            </geometry>
+        </visual>
+    </link>
+    <link name="gripper_left">
+        <visual>
+            <origin rpy="0 0 -${PI/2}" xyz="-0.04 0.5 -0.1"/>
+            <geometry>
+                <mesh filename="package://pickbot_description/meshes/left_finger.STL" scale="0.01 0.01 0.01"/>
+            </geometry>
+        </visual>
+    </link>
+    <joint name="joint_4" type="revolute">
+        <parent link="claw_support"/>
+        <child link="gripper_right"/>
+        <axis xyz="0 0 1"/>
+        <origin rpy="0 0 0" xyz="-0.04 0.13 -0.1"/>
+        <limit lower="-${PI/2}" upper="0.0" effort="${effort}" velocity="${velocity}"/>
+    </joint>
+    <joint name="joint_5" type="revolute">
+        <parent link="claw_support"/>
+        <child link="gripper_left"/>
+        <axis xyz="0 0 1"/>
+        <origin rpy="0 0 0" xyz="-0.22 0.13 -0.1"/>
+        <limit lower="0.0" upper="${PI/2}" effort="${effort}" velocity="${velocity}"/>
+        <mimic joint="joint_4" multiplier="-1"/>
+    </joint>
 </robot>

Commit message: added rgb camera to robot

File: pickbot_ws/install/pickbot_description/share/pickbot_description/urdf/pickbot.urdf.xacro (robot description, xacro)
@@ -107,3 +107,16 @@
         <mimic joint="joint_4" multiplier="-1"/>
     </joint>
+    <link name="rgb_camera">
+    <visual>
+        <origin rpy="-${PI/2} 0 -${PI/2}" xyz="-0.1 0.5 0.15"/>
+        <geometry>
+            <mesh filename="package://pickbot_description/meshes/pi_camera.STL" scale="0.01 0.01 0.01"/>
+        </geometry>
+    </visual>
+    </link>
+    <joint name="rgb_camera_joint" type="fixed">
+        <parent link="base_link"/>
+        <child link="rgb_camera"/>
+        <origin rpy="0 -0.5 ${PI/2}" xyz="0 0.45 0.2" />
+    </joint>
 </robot>

File: pickbot_ws/src/pickbot_description/urdf/pickbot.urdf.xacro (robot description, xacro)
@@ -107,3 +107,16 @@
         <mimic joint="joint_4" multiplier="-1"/>
     </joint>
+    <link name="rgb_camera">
+    <visual>
+        <origin rpy="-${PI/2} 0 -${PI/2}" xyz="-0.1 0.125 0.15"/>
+        <geometry>
+            <mesh filename="package://pickbot_description/meshes/pi_camera.STL" scale="0.01 0.01 0.01"/>
+        </geometry>
+    </visual>
+    </link>
+    <joint name="rgb_camera_joint" type="fixed">
+        <parent link="base_link"/>
+        <child link="rgb_camera"/>
+        <origin rpy="0 -0.5 ${PI/2}" xyz="0 0.45 0.2" />
+    </joint>
 </robot>

Commit message: added collision tag to urdf for simulation is gazebo

File: pickbot_ws/install/pickbot_description/share/pickbot_description/urdf/pickbot.urdf.xacro (robot description, xacro)
@@ -12,4 +12,10 @@
             </geometry>
         </visual>
+        <collision>
+            <origin rpy="0 0 0" xyz="-0.5 -0.5 0"/>
+            <geometry>
+                <mesh filename="package://pickbot_description/meshes/basement.STL" scale="0.01 0.01 0.01"/>
+            </geometry>
+        </collision>
     </link>
     <joint name="virtual_joint" type="fixed">
@@ -25,4 +31,10 @@
             </geometry>
         </visual>
+        <collision>
+            <origin rpy="0 0 0" xyz="-0.39 -0.39 -0.56"/>
+            <geometry>
+                <mesh filename="package://pickbot_description/meshes/base_plate.STL" scale="0.01 0.01 0.01"/>
+            </geometry>
+        </collision>
     </link>
     <joint name="joint_1" type="revolute">
@@ -40,4 +52,10 @@
             </geometry>
         </visual>
+        <collision>
+            <origin rpy="0 -${PI/2} ${PI/2}" xyz="0.19 0.06 -0.08"/>
+            <geometry>
+                <mesh filename="package://pickbot_description/meshes/forward_drive_arm.STL" scale="0.01 0.01 0.01"/>
+            </geometry>
+        </collision>
     </link>
     <joint name="joint_2" type="revolute">
@@ -55,4 +73,10 @@
             </geometry>
         </visual>
+        <collision>
+            <origin rpy="${PI/2} 0 ${PI/2}" xyz="-0.03 -0.4 -0.06"/>
+            <geometry>
+                <mesh filename="package://pickbot_description/meshes/horizontal_arm.STL" scale="0.01 0.01 0.01"/>
+            </geometry>
+        </collision>
     </link>
     <joint name="joint_3" type="revolute">
@@ -70,4 +94,10 @@
             </geometry>
         </visual>
+        <collision>
+            <origin rpy="0 0 ${PI/2}" xyz="0 -0.05 -0.15"/>
+            <geometry>
+                <mesh filename="package://pickbot_description/meshes/claw_support.STL" scale="0.01 0.01 0.01"/>
+            </geometry>
+        </collision>
     </link>
     <joint name="horizontal_arm_to_claw_support" type="fixed">
@@ -83,4 +113,10 @@
             </geometry>
         </visual>
+        <collision>
+            <origin rpy="0 0 -${PI/2}" xyz="-0.1 0.5 -0.1"/>
+            <geometry>
+                <mesh filename="package://pickbot_description/meshes/right_finger.STL" scale="0.01 0.01 0.01"/>
+            </geometry>
+        </collision>
     </link>
     <link name="gripper_left">
@@ -91,4 +127,10 @@
             </geometry>
         </visual>
+        <collision>
+            <origin rpy="0 0 -${PI/2}" xyz="-0.04 0.5 -0.1"/>
+            <geometry>
+                <mesh filename="package://pickbot_description/meshes/left_finger.STL" scale="0.01 0.01 0.01"/>
+            </geometry>
+        </collision>
     </link>
     <joint name="joint_4" type="revolute">
@@ -108,10 +150,16 @@
     </joint>
     <link name="rgb_camera">
-    <visual>
-        <origin rpy="-${PI/2} 0 -${PI/2}" xyz="-0.1 0.5 0.15"/>
-        <geometry>
-            <mesh filename="package://pickbot_description/meshes/pi_camera.STL" scale="0.01 0.01 0.01"/>
-        </geometry>
-    </visual>
+        <visual>
+            <origin rpy="-${PI/2} 0 -${PI/2}" xyz="-0.1 0.125 0.15"/>
+            <geometry>
+                <mesh filename="package://pickbot_description/meshes/pi_camera.STL" scale="0.01 0.01 0.01"/>
+            </geometry>
+        </visual>
+        <collision>
+            <origin rpy="-${PI/2} 0 -${PI/2}" xyz="-0.1 0.125 0.15"/>
+            <geometry>
+                <mesh filename="package://pickbot_description/meshes/pi_camera.STL" scale="0.01 0.01 0.01"/>
+            </geometry>
+        </collision>
     </link>
     <joint name="rgb_camera_joint" type="fixed">

File: pickbot_ws/src/pickbot_description/urdf/pickbot.urdf.xacro (robot description, xacro)
@@ -12,4 +12,10 @@
             </geometry>
         </visual>
+        <collision>
+            <origin rpy="0 0 0" xyz="-0.5 -0.5 0"/>
+            <geometry>
+                <mesh filename="package://pickbot_description/meshes/basement.STL" scale="0.01 0.01 0.01"/>
+            </geometry>
+        </collision>
     </link>
     <joint name="virtual_joint" type="fixed">
@@ -25,4 +31,10 @@
             </geometry>
         </visual>
+        <collision>
+            <origin rpy="0 0 0" xyz="-0.39 -0.39 -0.56"/>
+            <geometry>
+                <mesh filename="package://pickbot_description/meshes/base_plate.STL" scale="0.01 0.01 0.01"/>
+            </geometry>
+        </collision>
     </link>
     <joint name="joint_1" type="revolute">
@@ -40,4 +52,10 @@
             </geometry>
         </visual>
+        <collision>
+            <origin rpy="0 -${PI/2} ${PI/2}" xyz="0.19 0.06 -0.08"/>
+            <geometry>
+                <mesh filename="package://pickbot_description/meshes/forward_drive_arm.STL" scale="0.01 0.01 0.01"/>
+            </geometry>
+        </collision>
     </link>
     <joint name="joint_2" type="revolute">
@@ -55,4 +73,10 @@
             </geometry>
         </visual>
+        <collision>
+            <origin rpy="${PI/2} 0 ${PI/2}" xyz="-0.03 -0.4 -0.06"/>
+            <geometry>
+                <mesh filename="package://pickbot_description/meshes/horizontal_arm.STL" scale="0.01 0.01 0.01"/>
+            </geometry>
+        </collision>
     </link>
     <joint name="joint_3" type="revolute">
@@ -70,4 +94,10 @@
             </geometry>
         </visual>
+        <collision>
+            <origin rpy="0 0 ${PI/2}" xyz="0 -0.05 -0.15"/>
+            <geometry>
+                <mesh filename="package://pickbot_description/meshes/claw_support.STL" scale="0.01 0.01 0.01"/>
+            </geometry>
+        </collision>
     </link>
     <joint name="horizontal_arm_to_claw_support" type="fixed">
@@ -83,4 +113,10 @@
             </geometry>
         </visual>
+        <collision>
+            <origin rpy="0 0 -${PI/2}" xyz="-0.1 0.5 -0.1"/>
+            <geometry>
+                <mesh filename="package://pickbot_description/meshes/right_finger.STL" scale="0.01 0.01 0.01"/>
+            </geometry>
+        </collision>
     </link>
     <link name="gripper_left">
@@ -91,4 +127,10 @@
             </geometry>
         </visual>
+        <collision>
+            <origin rpy="0 0 -${PI/2}" xyz="-0.04 0.5 -0.1"/>
+            <geometry>
+                <mesh filename="package://pickbot_description/meshes/left_finger.STL" scale="0.01 0.01 0.01"/>
+            </geometry>
+        </collision>
     </link>
     <joint name="joint_4" type="revolute">
@@ -108,10 +150,16 @@
     </joint>
     <link name="rgb_camera">
-    <visual>
-        <origin rpy="-${PI/2} 0 -${PI/2}" xyz="-0.1 0.125 0.15"/>
-        <geometry>
-            <mesh filename="package://pickbot_description/meshes/pi_camera.STL" scale="0.01 0.01 0.01"/>
-        </geometry>
-    </visual>
+        <visual>
+            <origin rpy="-${PI/2} 0 -${PI/2}" xyz="-0.1 0.125 0.15"/>
+            <geometry>
+                <mesh filename="package://pickbot_description/meshes/pi_camera.STL" scale="0.01 0.01 0.01"/>
+            </geometry>
+        </visual>
+        <collision>
+            <origin rpy="-${PI/2} 0 -${PI/2}" xyz="-0.1 0.125 0.15"/>
+            <geometry>
+                <mesh filename="package://pickbot_description/meshes/pi_camera.STL" scale="0.01 0.01 0.01"/>
+            </geometry>
+        </collision>
     </link>
     <joint name="rgb_camera_joint" type="fixed">

Commit message: added launch file to simulate robot in gazebo

File: pickbot_ws/install/pickbot_description/share/pickbot_description/urdf/pickbot.urdf.xacro (robot description, xacro)
@@ -4,6 +4,16 @@
     <xacro:property name="effort" value="30.0"/>
     <xacro:property name="velocity" value="10.0"/>
+    <xacro:macro name="default_inertial" params="mass">
+        <inertial>
+            <origin xyz="0 0 0" rpy="0 0 0"/>
+            <mass value="${mass}" />
+            <inertia ixx="1.0" ixy="0.0" ixz="0.0"
+                    iyy="1.0" iyz="0.0"
+                    izz="1.0"/>
+        </inertial>
+    </xacro:macro>
     <link name="world"/>
     <link name="base_link">
+        <xacro:default_inertial mass="1.0"/>
         <visual>
             <origin rpy="0 0 0" xyz="-0.5 -0.5 0"/>
@@ -25,4 +35,5 @@
     </joint>
     <link name="base_plate">
+        <xacro:default_inertial mass="0.1"/>
         <visual>
             <origin rpy="0 0 0" xyz="-0.39 -0.39 -0.56"/>
@@ -46,4 +57,5 @@
     </joint>
     <link name="forward_drive_arm">
+        <xacro:default_inertial mass="0.1"/>
         <visual>
             <origin rpy="0 -${PI/2} ${PI/2}" xyz="0.19 0.06 -0.08"/>
@@ -67,4 +79,5 @@
     </joint>
     <link name="horizontal_arm">
+        <xacro:default_inertial mass="0.1"/>
         <visual>
             <origin rpy="${PI/2} 0 ${PI/2}" xyz="-0.03 -0.4 -0.06"/>
@@ -88,4 +101,5 @@
     </joint>
     <link name="claw_support">
+        <xacro:default_inertial mass="0.05"/>
         <visual>
             <origin rpy="0 0 ${PI/2}" xyz="0 -0.05 -0.15"/>
@@ -107,4 +121,5 @@
     </joint>
     <link name="gripper_right">
+        <xacro:default_inertial mass="0.01"/>
         <visual>
             <origin rpy="0 0 -${PI/2}" xyz="-0.1 0.5 -0.1"/>
@@ -121,4 +136,5 @@
     </link>
     <link name="gripper_left">
+        <xacro:default_inertial mass="0.01"/>
         <visual>
             <origin rpy="0 0 -${PI/2}" xyz="-0.04 0.5 -0.1"/>

File: pickbot_ws/src/pickbot_description/urdf/pickbot.urdf.xacro (robot description, xacro)
@@ -6,7 +6,8 @@
     <xacro:macro name="default_inertial" params="mass">
         <inertial>
-            <mass value="${mass}"/>
-            <inertia ixx="1.0" ixy="1.0" ixz="1.0"
-                    iyy="1.0" iyz="1.0"
+            <origin xyz="0 0 0" rpy="0 0 0"/>
+            <mass value="${mass}" />
+            <inertia ixx="1.0" ixy="0.0" ixz="0.0"
+                    iyy="1.0" iyz="0.0"
                     izz="1.0"/>
         </inertial>
